Commit message: adding veehicle description support

File: src/autoware.AI/visualization/vehicle_description/urdf/vehicleB_lexus.urdf (robot description, URDF)
Before this commit: robot car, 1 links, 0 joints
Links:
- removed link base_link
- added link vehicleB_base_link; visual mesh filename=package://vehicle_description/mesh/lexus.dae scale=1.0 1.0 1.0
